Commit message: add room

File: aubo_description/urdf/aubo_i5.urdf.xacro (robot description, xacro)
@@ -204,9 +204,71 @@
     <limit lower="-3.05" upper="3.05" effort="0" velocity="0" />
   </joint>
-  <link name="world" />
+  <!-- <link name="world" />
   <joint name="world_joint" type="fixed">
     <parent link="world" />
     <child link = "base_link" />
     <origin xyz="0.0 0.0 0.0" rpy="0.0 0.0 0.0" />
-  </joint>
+  </joint> -->
+<!-- /////////////////////////////////   i5 coonection link   ////////////////////////////////////// -->
+  <link name="connect_Link">
+    <visual>
+      <geometry>
+        <mesh filename="package://aubo_description/meshes/aubo_i5/visual/connect_robo.STL" />
+      </geometry>
+    </visual>
+  </link>
+  <joint name="connect_joint" type="fixed">
+    <parent link="connect_Link"/>
+    <child link="base_link"/>
+    <origin xyz="0 0 0" rpy="0 0 0" />
+  </joint>
+  <!-- /////////////////////////////////   i5 room_Link   ////////////////////////////////////// -->
+  <link name="room_Link">
+    <visual>
+      <geometry>
+        <mesh filename="package://aubo_description/meshes/aubo_i5/visual/env.STL" scale="0.001 0.001 0.001" />
+      </geometry>
+    </visual>
+  </link>
+  <joint name="room_joint" type="fixed">
+    <parent link="room_Link"/>
+    <child link="connect_Link"/>
+    <origin xyz="0 0 0" rpy="1.5708 0 3.1415926" />
+  </joint>
+ <!-- /////////////////////////////////   world   ////////////////////////////////////// -->
+  <link name="world" />
+  <joint name="world_joint" type="fixed">
+    <parent link="world" />
+    <child link ="room_Link" />
+    <origin xyz="0.0 0.0 6.0" rpy="1.5708 0.0 2.1416" />
+  </joint>
+  <!-- /////////////////////////////////   gazebo color   ////////////////////////////////////// -->
+  <gazebo reference="room_Link">
+     <material>Gazebo/Grey</material>
+  </gazebo>
+  <!--////////////////////////////////// Transmissions for ROS Control //////////////////////////-->
+<xacro:macro name="aubo_arm_transmission" params="joint_name">
+     <transmission name="${joint_name}_trans">
+       <type>transmission_interface/SimpleTransmission</type>
+       <joint name="${joint_name}">
+         <!--<hardwareInterface>hardware_interface/PositionJointInterface</hardwareInterface>-->
+         <hardwareInterface>hardware_interface/PositionJointInterface</hardwareInterface>
+       </joint>
+       <actuator name="${joint_name}_motor">
+         <mechanicalReduction>1</mechanicalReduction>
+       </actuator>
+     </transmission>
+ </xacro:macro>
+  <xacro:aubo_arm_transmission joint_name="shoulder_joint"/>
+  <xacro:aubo_arm_transmission joint_name="upperArm_joint"/>
+  <xacro:aubo_arm_transmission joint_name="foreArm_joint"/>
+  <xacro:aubo_arm_transmission joint_name="wrist1_joint"/>
+  <xacro:aubo_arm_transmission joint_name="wrist2_joint"/>
+  <xacro:aubo_arm_transmission joint_name="wrist3_joint"/>
+  <!-- ros_control plugin -->
+  <gazebo>
+      <plugin name="gazebo_ros_control" filename="libgazebo_ros_control.so">
+          <robotNamespace>/aubo_i5</robotNamespace>
+      </plugin>
+  </gazebo>
 </robot>

Commit message: room ready, need to add supporter for robot

File: aubo_description/urdf/aubo_i5.urdf.xacro (robot description, xacro)
@@ -241,5 +241,5 @@
     <parent link="world" />
     <child link ="room_Link" />
-    <origin xyz="0.0 0.0 6.0" rpy="1.5708 0.0 2.1416" />
+    <origin xyz="0.0 0.0 0.0" rpy="1.5708 0.0 3.1416" />
   </joint>
   <!-- /////////////////////////////////   gazebo color   ////////////////////////////////////// -->

Commit message: add connector for aubo

File: aubo_description/urdf/aubo_i5.urdf.xacro (robot description, xacro)
@@ -30,5 +30,5 @@
     </collision>
   </link>
-  <link name="shoulder_Link">
+  <!-- <link name="shoulder_Link">
     <inertial>
       <origin xyz="3.2508868974735E-07 0.00534955349296065 -0.00883689325611056" rpy="0 0 0" />
@@ -203,5 +203,5 @@
     <axis xyz="0 0 1" />
     <limit lower="-3.05" upper="3.05" effort="0" velocity="0" />
-  </joint>
+  </joint> -->
   <!-- <link name="world" />
   <joint name="world_joint" type="fixed">
@@ -214,5 +214,5 @@
     <visual>
       <geometry>
-        <mesh filename="package://aubo_description/meshes/aubo_i5/visual/connect_robo.STL" />
+        <mesh filename="package://aubo_description/meshes/aubo_i5/visual/connect_robo.STL" scale="0.001 0.001 0.001" />
       </geometry>
     </visual>
@@ -221,5 +221,5 @@
     <parent link="connect_Link"/>
     <child link="base_link"/>
-    <origin xyz="0 0 0" rpy="0 0 0" />
+    <origin xyz="0.17 0.085 -0.0" rpy="3.1415926 0 0" />
   </joint>
   <!-- /////////////////////////////////   i5 room_Link   ////////////////////////////////////// -->
@@ -234,5 +234,5 @@
     <parent link="room_Link"/>
     <child link="connect_Link"/>
-    <origin xyz="0 0 0" rpy="1.5708 0 3.1415926" />
+    <origin xyz="4 1.77 0.0" rpy="1.5708 0 3.1415926" />
   </joint>
  <!-- /////////////////////////////////   world   ////////////////////////////////////// -->
@@ -260,5 +260,5 @@
      </transmission>
  </xacro:macro>
-  <xacro:aubo_arm_transmission joint_name="shoulder_joint"/>
+  <!-- <xacro:aubo_arm_transmission joint_name="shoulder_joint"/>
   <xacro:aubo_arm_transmission joint_name="upperArm_joint"/>
   <xacro:aubo_arm_transmission joint_name="foreArm_joint"/>
@@ -266,4 +266,5 @@
   <xacro:aubo_arm_transmission joint_name="wrist2_joint"/>
   <xacro:aubo_arm_transmission joint_name="wrist3_joint"/>
+ -->
   <!-- ros_control plugin -->
   <gazebo>

Commit message: add car inside room

File: aubo_description/urdf/aubo_i5.urdf.xacro (robot description, xacro)
@@ -30,5 +30,5 @@
     </collision>
   </link>
-  <!-- <link name="shoulder_Link">
+  <link name="shoulder_Link">
     <inertial>
       <origin xyz="3.2508868974735E-07 0.00534955349296065 -0.00883689325611056" rpy="0 0 0" />
@@ -203,11 +203,5 @@
     <axis xyz="0 0 1" />
     <limit lower="-3.05" upper="3.05" effort="0" velocity="0" />
-  </joint> -->
-  <!-- <link name="world" />
-  <joint name="world_joint" type="fixed">
-    <parent link="world" />
-    <child link = "base_link" />
-    <origin xyz="0.0 0.0 0.0" rpy="0.0 0.0 0.0" />
-  </joint> -->
+  </joint>
 <!-- /////////////////////////////////   i5 coonection link   ////////////////////////////////////// -->
   <link name="connect_Link">
@@ -231,4 +225,11 @@
     </visual>
   </link>
+  <link name="car_Link">
+    <visual>
+      <geometry>
+        <mesh filename="package://aubo_description/meshes/aubo_i5/visual/car.stl" scale="0.001 0.001 0.001" />
+      </geometry>
+    </visual>
+  </link>
   <joint name="room_joint" type="fixed">
     <parent link="room_Link"/>
@@ -238,12 +239,30 @@
  <!-- /////////////////////////////////   world   ////////////////////////////////////// -->
   <link name="world" />
-  <joint name="world_joint" type="fixed">
-    <parent link="world" />
+  <link name="link0" />
+    <joint name="world_joint" type="fixed">
+      <parent link="world" />
+      <child link="link0" />
+      <origin xyz="0 0 0" rpy="0 0 0"/>
+      <axis xyz="0 0 1"/>
+    </joint>
+  <joint name="wash_joint" type="fixed">
+    <parent link="link0" />
     <child link ="room_Link" />
     <origin xyz="0.0 0.0 0.0" rpy="1.5708 0.0 3.1416" />
   </joint>
+  <joint name="car_joint" type="fixed">
+    <parent link="link0" />
+    <child link ="car_Link" />
+    <origin xyz="-3 0.0 0.0" rpy="0 0.0 0" />
+  </joint>
   <!-- /////////////////////////////////   gazebo color   ////////////////////////////////////// -->
+  <gazebo reference="car_Link">
+     <material>Gazebo/Green</material>
+  </gazebo>
   <gazebo reference="room_Link">
-     <material>Gazebo/Grey</material>
+     <material>Gazebo/Blue</material>
+  </gazebo>
+   <gazebo reference="connect_Link">
+     <material>Gazebo/Black</material>
   </gazebo>
   <!--////////////////////////////////// Transmissions for ROS Control //////////////////////////-->
@@ -260,5 +279,5 @@
      </transmission>
  </xacro:macro>
-  <!-- <xacro:aubo_arm_transmission joint_name="shoulder_joint"/>
+  <xacro:aubo_arm_transmission joint_name="shoulder_joint"/>
   <xacro:aubo_arm_transmission joint_name="upperArm_joint"/>
   <xacro:aubo_arm_transmission joint_name="foreArm_joint"/>
@@ -266,5 +285,4 @@
   <xacro:aubo_arm_transmission joint_name="wrist2_joint"/>
   <xacro:aubo_arm_transmission joint_name="wrist3_joint"/>
- -->
   <!-- ros_control plugin -->
   <gazebo>
